File: kicad/usb-c_demo1/usb-c_demo1.kicad_pcb (KiCad board)
At the start: 2 copper layers, 45.7 x 33 mm, 34 parts, among them J1 USB_C_Receptacle_USB2.0, J2 SWD, J3 Screw_Terminal_01x03, J4 Conn_01x06, J5 Conn_01x06, U1 STM32G431KBT6, U2 USBLC6-2SC6, U7 MIC5317-3.3YM5-TR, Y1 16MHz

Commit message: routing
Parts:
- J3: value Screw_Terminal_01x03 -> LED
- R2: footprint Resistor_SMD:R_0603_1608Metric_Pad0.98x0.95mm_HandSolder -> Resistor_SMD:R_0603_1608Metric
- moved R2 26.3 mm to (36.1, 47.2)
- moved R3 22.6 mm to (38.4, 47.2)
- moved D1 21.7 mm to (36.1, 51.1), turned to -90 degrees
- moved D2 19.1 mm to (38.4, 51.1), turned to -90 degrees
- moved FB1 10.7 mm to (70.4, 54.9), turned to 90 degrees
- moved F1 8.03 mm to (66.8, 54.9)
- moved C8 7.25 mm to (62.0, 54.2), turned to 0 degrees
- moved C6 6.27 mm to (47.5, 70.9), turned to -90 degrees
- moved C9 6.11 mm to (62.0, 47.9), turned to 0 degrees
- moved C7 5.66 mm to (49.5, 70.9), turned to -90 degrees
- moved U7 4.97 mm to (62.0, 51.1), turned to 90 degrees
- moved C3 3.98 mm to (55.1, 68.3)
- moved R4 3.61 mm to (35.8, 56.1)
- moved C4 1.85 mm to (39.9, 60.2)
- moved C1 1.85 mm to (35.8, 58.2)
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Connections:
- net Net-(R4-Pad1) renamed /BOOT0
- J1 pad S1: /SHIELD -> unconnected-(J1-PadS1)
- J4 pad 1: unconnected-(J4-Pad1) -> GND
- J4 pad 2: unconnected-(J4-Pad2) -> +3V3
- J4 pad 3: unconnected-(J4-Pad3) -> PA4
- J4 pad 4: unconnected-(J4-Pad4) -> PA5
- J4 pad 5: unconnected-(J4-Pad5) -> PA6
- J4 pad 6: unconnected-(J4-Pad6) -> PA7
- J5 pad 1: unconnected-(J5-Pad1) -> GND
- J5 pad 2: unconnected-(J5-Pad2) -> +3V3
- J5 pad 3: unconnected-(J5-Pad3) -> PA0
- J5 pad 4: unconnected-(J5-Pad4) -> PA1
- J5 pad 5: unconnected-(J5-Pad5) -> PA2
- J5 pad 6: unconnected-(J5-Pad6) -> PA3
- U1 pad 10: unconnected-(U1-Pad10) -> PA5
- U1 pad 11: unconnected-(U1-Pad11) -> PA6
- U1 pad 12: unconnected-(U1-Pad12) -> PA7
- U1 pad 30: unconnected-(U1-Pad30) -> STATUS_LED
- U1 pad 5: unconnected-(U1-Pad5) -> PA0
- U1 pad 6: unconnected-(U1-Pad6) -> PA1
- U1 pad 7: unconnected-(U1-Pad7) -> PA2
- U1 pad 8: unconnected-(U1-Pad8) -> PA3
- U1 pad 9: unconnected-(U1-Pad9) -> PA4
Routing:
- net /VBUS: track 0.00 -> 43.6 mm, vias 0 -> 2
- net GND: track 0.00 -> 28.3 mm, vias 0 -> 38
- net NRST: track 0.00 -> 27.7 mm, vias 0 -> 2
- net PA0: track 0.00 -> 22.4 mm
- net PA1: track 0.00 -> 19.7 mm
- net PA2: track 0.00 -> 19.1 mm
- net +3V3: track 0.00 -> 18.3 mm, vias 0 -> 10
- net PA3: track 0.00 -> 18.1 mm
- net +5V: track 0.00 -> 15.2 mm
- net STATUS_LED: track 0.00 -> 13.7 mm
- net PIXEL: track 0.00 -> 13.0 mm, vias 0 -> 1
- net /OSC_IN: track 0.00 -> 11.5 mm
- net /BOOT0: track 0.00 -> 11.4 mm
- net SWDIO: track 0.00 -> 11.3 mm
- net SWCLK: track 0.00 -> 9.52 mm
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- added copper zone on In2.Cu, net +3V3
- added copper zone on F.Cu, net /VBUS
- added copper zone on B.Cu, net GND
- added copper zone on F.Cu, net GND
- added copper zone on In1.Cu, net GND
Other:
- copper layers 2 -> 4
- board text added: "+"
- board text added: "-"
- board text added: "JLCJLCJLCJLC"
- board text added: "Laurent Fiack 2022"
- board text added: "P"
- board text added: "PA0"
- board text added: "PA1"
- board text added: "PA2"
- board text added: "PA3"
- board text added: "PA4"
- board text added: "PA5"
- board text added: "PA6"
- board text added: "PA7"
- board text added: "PIX"
- board text added: "S"
- board text added: "USB-C Demo STM32G431KBT6 Rev 1.0"
