File: kicad/usb-c_demo1/usb-c_demo1.kicad_sch (KiCad schematic)
At the start: 34 parts, among them J1 USB_C_Receptacle_USB2.0, J2 SWD, J3 Screw_Terminal_01x03, J4 Conn_01x06, J5 Conn_01x06, U1 STM32G431KBT6, U2 USBLC6-2SC6, U7 MIC5317-3.3YM5-TR, Y1 16MHz

Commit message: routing
Parts:
- R2: footprint Resistor_SMD:R_0603_1608Metric_Pad0.98x0.95mm_HandSolder -> Resistor_SMD:R_0603_1608Metric
Connections:
- net +3V3: now also J4.2 (Pin_2), J5.2 (Pin_2)
- net GND: now also J4.1 (Pin_1), J5.1 (Pin_1)
- net STATUS_LED: now also U1.30 (PB7)
- net PA5: now reaches U1.10 (PA5)
- net PA5: now also J4.4 (Pin_4)
- net PA6: now reaches U1.11 (PA6)
- net PA6: now also J4.5 (Pin_5)
- net PA7: now reaches U1.12 (PA7)
- net PA7: now also J4.6 (Pin_6)
- net BOOT0: now reaches R4.1, U1.31 (PB8-BOOT)
- net PA0: now reaches U1.5 (PA0)
- net PA0: now also J5.3 (Pin_3)
- net PA1: now reaches U1.6 (PA1)
- net PA1: now also J5.4 (Pin_4)
- net PA2: now reaches U1.7 (PA2)
- net PA2: now also J5.5 (Pin_5)
- net PA3: now reaches U1.8 (PA3)
- net PA3: now also J5.6 (Pin_6)
- net PA4: now reaches U1.9 (PA4)
- net PA4: now also J4.3 (Pin_3)
- net SHIELD: no longer names the net of J1.S1 (SHIELD)
- no-connect marks 3 -> 10
Other:
- moved on the sheet: J5, R4
